File: Dinkydox.sch (KiCad schematic (older format))
At the start: 47 parts, among them K1 KEYSW, K10 KEYSW, K11 KEYSW, K12 KEYSW, K13 KEYSW, K14 KEYSW, K15 KEYSW, K16 KEYSW, K17 KEYSW, K18 KEYSW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

Commit message: Rename 6col
Parts:
- D1, D10, D11, D12, D13, D14, D15, D16, D17, D18, D19, D2, D20, D21, D3, D4, D5, D6, D7, D8, D9: symbol Device:D -> 6col-rescue:D-Device
- K1, K10, K11, K12, K13, K14, K15, K16, K17, K18, K19, K2, K20, K21, K3, K4, K5, K6, K7, K8, K9: symbol canadian_parts:KEYSW -> 6col-rescue:KEYSW-canadian_parts
- K22: symbol canadian_parts:TRRS_Through-Hole -> 6col-rescue:TRRS_Through-Hole-canadian_parts
- RESET1: symbol keyboard_parts:SW_PUSH -> 6col-rescue:SW_PUSH-keyboard_parts
- SJ1, SJ2: symbol canadian_parts:SOLDER_JUMPER_3 -> 6col-rescue:SOLDER_JUMPER_3-canadian_parts
- U1: symbol ProMicro:ProMicro -> 6col-rescue:ProMicro-ProMicro
Changed lines of the file:
@@
 $EndDescr
 $Comp
-L canadian_parts:KEYSW K1
+L 6col-rescue:KEYSW-canadian_parts K1
 U 1 1 588E249B
 P 2300 1950
@@
 $EndComp
 $Comp
-L Device:D D2
+L 6col-rescue:D-Device D2
 U 1 1 588E259A
 P 2800 2200
@@
 $EndComp
 $Comp
-L canadian_parts:KEYSW K2
+L 6col-rescue:KEYSW-canadian_parts K2
 U 1 1 588E266D
 P 3200 1950
@@
 $EndComp
 $Comp
-L canadian_parts:KEYSW K3
+L 6col-rescue:KEYSW-canadian_parts K3
 U 1 1 588E26B1
 P 4100 1950
@@
 $EndComp
 $Comp
-L canadian_parts:KEYSW K4
+L 6col-rescue:KEYSW-canadian_parts K4
 U 1 1 588E271C
 P 5000 1950
@@
 $EndComp
 $Comp
-L Device:D D1
+L 6col-rescue:D-Device D1
 U 1 1 588E27E6
 P 1900 2200
@@
 $EndComp
 $Comp
-L Device:D D3
+L 6col-rescue:D-Device D3
 U 1 1 588E28C6
 P 3700 2200
@@
 $EndComp
 $Comp
-L Device:D D4
+L 6col-rescue:D-Device D4
 U 1 1 588E2919
 P 4600 2200
@@
 $EndComp
 $Comp
-L canadian_parts:KEYSW K7
+L 6col-rescue:KEYSW-canadian_parts K7
 U 1 1 588E2B6A
 P 2300 2550
@@
 $EndComp
 $Comp
-L Device:D D8
+L 6col-rescue:D-Device D8
 U 1 1 588E2B70
 P 2800 2800
@@
 $EndComp
 $Comp
-L canadian_parts:KEYSW K8
+L 6col-rescue:KEYSW-canadian_parts K8
 U 1 1 588E2B76
 P 3200 2550
@@
 $EndComp
 $Comp
-L canadian_parts:KEYSW K9
+L 6col-rescue:KEYSW-canadian_parts K9
 U 1 1 588E2B7C
 P 4100 2550
@@
 $EndComp
 $Comp
-L canadian_parts:KEYSW K10
+L 6col-rescue:KEYSW-canadian_parts K10
 U 1 1 588E2B82
 P 5000 2550
@@
 $EndComp
 $Comp
-L Device:D D7
+L 6col-rescue:D-Device D7
 U 1 1 588E2B8E
 P 1900 2800
@@
 $EndComp
 $Comp
-L Device:D D9
+L 6col-rescue:D-Device D9
 U 1 1 588E2B94
 P 3700 2800
@@
 $EndComp
 $Comp
-L canadian_parts:KEYSW K13
+L 6col-rescue:KEYSW-canadian_parts K13
 U 1 1 588E2DFE
 P 2300 3150
@@
 $EndComp
 $Comp
-L Device:D D14
+L 6col-rescue:D-Device D14
 U 1 1 588E2E04
 P 2800 3400
@@
 $EndComp
 $Comp
-L canadian_parts:KEYSW K14
+L 6col-rescue:KEYSW-canadian_parts K14
 U 1 1 588E2E0A
 P 3200 3150
@@
 $EndComp
 $Comp
-L canadian_parts:KEYSW K15
+L 6col-rescue:KEYSW-canadian_parts K15
 U 1 1 588E2E10
 P 4100 3150
@@
 $EndComp
 $Comp
-L canadian_parts:KEYSW K16
+L 6col-rescue:KEYSW-canadian_parts K16
 U 1 1 588E2E16
 P 5000 3150
@@
 $EndComp
 $Comp
-L Device:D D15
+L 6col-rescue:D-Device D15
 U 1 1 588E2E28
 P 3700 3400
@@
 $EndComp
 $Comp
-L Device:D D16
+L 6col-rescue:D-Device D16
 U 1 1 588E2E2E
 P 4600 3400
@@
 $EndComp
 $Comp
-L canadian_parts:KEYSW K19
+L 6col-rescue:KEYSW-canadian_parts K19
 U 1 1 588E314C
 P 5000 3750
@@
 $EndComp
 $Comp
-L Device:D D19
+L 6col-rescue:D-Device D19
 U 1 1 588E315E
 P 4600 4000
@@
 $EndComp
 $Comp
-L canadian_parts:SOLDER_JUMPER_3 SJ2
+L 6col-rescue:SOLDER_JUMPER_3-canadian_parts SJ2
 U 1 1 588E8D2F
 P 7900 2300
@@
 $EndComp
 $Comp
-L canadian_parts:SOLDER_JUMPER_3 SJ1
+L 6col-rescue:SOLDER_JUMPER_3-canadian_parts SJ1
 U 1 1 588E912F
 P 8450 1850
@@
 $EndComp
 $Comp
-L power:GND #PWR01
+L 6col-rescue:GND-power #PWR01
 U 1 1 588EB154
 P 8700 1800
@@
 $EndComp
 $Comp
-L power:GND #PWR02
+L 6col-rescue:GND-power #PWR02
 U 1 1 588EB1B8
 P 8150 2250
@@
 $EndComp
 $Comp
-L power:GND #PWR03
+L 6col-rescue:GND-power #PWR03
 U 1 1 588EB71C
 P 8800 4400
@@
 $EndComp
 $Comp
-L power:GND #PWR04
+L 6col-rescue:GND-power #PWR04
 U 1 1 588EB780
 P 7800 4600
@@
 $EndComp
 $Comp
-L power:GND #PWR05
+L 6col-rescue:GND-power #PWR05
 U 1 1 588EB7E4
 P 7800 4500
@@
 $EndComp
 $Comp
-L power:VCC #PWR06
+L 6col-rescue:VCC-power #PWR06
 U 1 1 588EB848
 P 8800 4600
@@
 $EndComp
 $Comp
-L power:VCC #PWR07
+L 6col-rescue:VCC-power #PWR07
 U 1 1 588EBC1C
 P 8350 1800
@@
 $EndComp
 $Comp
-L power:VCC #PWR08
+L 6col-rescue:VCC-power #PWR08
 U 1 1 588EBC80
 P 7800 2250
@@
 data
 $Comp
-L keyboard_parts:SW_PUSH RESET1
+L 6col-rescue:SW_PUSH-keyboard_parts RESET1
 U 1 1 588F2D74
 P 9400 4500
@@
 $EndComp
 $Comp
-L power:GND #PWR09
+L 6col-rescue:GND-power #PWR09
 U 1 1 588F2E25
 P 9700 4500
@@
 $EndComp
 $Comp
-L Device:D D13
+L 6col-rescue:D-Device D13
 U 1 1 588E2E22
 P 1900 3400
@@
 $EndComp
 $Comp
-L Device:D D10
+L 6col-rescue:D-Device D10
 U 1 1 588E2B9A
 P 4600 2800
@@
 $EndComp
 $Comp
-L Device:D D20
+L 6col-rescue:D-Device D20
 U 1 1 588E3164
 P 5500 4000
@@
 $EndComp
 $Comp
-L canadian_parts:KEYSW K20
+L 6col-rescue:KEYSW-canadian_parts K20
 U 1 1 588E3152
 P 5900 3750
@@
 $EndComp
 $Comp
-L Device:D D17
+L 6col-rescue:D-Device D17
 U 1 1 588E2E34
 P 5500 3400
@@
 $EndComp
 $Comp
-L canadian_parts:KEYSW K17
+L 6col-rescue:KEYSW-canadian_parts K17
 U 1 1 588E2E1C
 P 5900 3150
@@
 $EndComp
 $Comp
-L Device:D D11
+L 6col-rescue:D-Device D11
 U 1 1 588E2BA0
 P 5500 2800
@@
 $EndComp
 $Comp
-L canadian_parts:KEYSW K11
+L 6col-rescue:KEYSW-canadian_parts K11
 U 1 1 588E2B88
 P 5900 2550
@@
 $EndComp
 $Comp
-L Device:D D5
+L 6col-rescue:D-Device D5
 U 1 1 588E2967
 P 5500 2200
@@
 $EndComp
 $Comp
-L canadian_parts:KEYSW K5
+L 6col-rescue:KEYSW-canadian_parts K5
 U 1 1 588E275E
 P 5900 1950
@@
 $EndComp
 $Comp
-L Device:D D21
+L 6col-rescue:D-Device D21
 U 1 1 5E2DC50C
 P 6450 4000
@@
 $EndComp
 $Comp
-L canadian_parts:KEYSW K21
+L 6col-rescue:KEYSW-canadian_parts K21
 U 1 1 5E2DC512
 P 6850 3750
@@
 $EndComp
 $Comp
-L Device:D D18
+L 6col-rescue:D-Device D18
 U 1 1 5E2DC518
 P 6450 3400
@@
 $EndComp
 $Comp
-L canadian_parts:KEYSW K18
+L 6col-rescue:KEYSW-canadian_parts K18
 U 1 1 5E2DC51E
 P 6850 3150
@@
 $EndComp
 $Comp
-L Device:D D12
+L 6col-rescue:D-Device D12
 U 1 1 5E2DC524
 P 6450 2800
@@
 $EndComp
 $Comp
-L canadian_parts:KEYSW K12
+L 6col-rescue:KEYSW-canadian_parts K12
 U 1 1 5E2DC52A
 P 6850 2550
@@
 $EndComp
 $Comp
-L Device:D D6
+L 6col-rescue:D-Device D6
 U 1 1 5E2DC530
 P 6450 2200
@@
 $EndComp
 $Comp
-L canadian_parts:KEYSW K6
+L 6col-rescue:KEYSW-canadian_parts K6
 U 1 1 5E2DC536
 P 6850 1950
@@
 $EndComp
 $Comp
-L canadian_parts:TRRS_Through-Hole K22
+L 6col-rescue:TRRS_Through-Hole-canadian_parts K22
 U 1 1 588E654E
 P 8550 2450
@@
 $EndComp
 $Comp
-L ProMicro:ProMicro U1
+L 6col-rescue:ProMicro-ProMicro U1
 U 1 1 588E2344
 P 8300 4650
